Commit message: new URDF

File: urdf/rosmower.xacro (robot description, xacro)
@@ -67,5 +67,5 @@
   </link>
   <joint name="base_link_joint" type="fixed">
-    <origin xyz="0 0 ${wheel_radius + 0.005}" rpy="0 0 0" />
+    <origin xyz="0.14 0 ${wheel_radius + 0.005}" rpy="0 0 0" />
     <parent link="base_footprint"/>
     <child link="base_link" />
@@ -134,13 +134,13 @@
     <parent link="base_link" />
     <child link="imu" />
-    <origin xyz="0.16 -0.065 0.035" rpy="0 0 0" />
+    <origin xyz="0.157 0.0 0.20" rpy="0 0 0" />
   </joint>
   <link name="imu" />
   <joint name="lidar_joint" type="fixed">
     <parent link="base_link" />
-    <child link="lidar" />
-    <origin xyz="0.0 0.0 0.12" rpy="0 0 3.14159" />
+    <child link="lidar_frame" />
+    <origin xyz="0.157 0.0 0.21" rpy="0 0 0" />
   </joint>
-  <link name="lidar">
+  <link name="lidar_frame">
     <visual>
       <material name="blue" />

Commit message: ekf pose package added

File: urdf/rosmower.xacro (robot description, xacro)
@@ -37,5 +37,4 @@
     </inertial>
   </xacro:macro>
-  <link name="dummy"/>
   <link name="base_footprint">
     <xacro:box_inertia m="8" w="0.001" h="0.001" d="0.001"/>
@@ -48,8 +47,4 @@
     </visual>
   </link>
-  <joint name="dummy_joint" type="fixed">
-     <parent link="dummy"/>
-     <child link="base_footprint"/>
-     </joint>
   <link name="base_link">
     <xacro:box_inertia m="1" w="${base_len}" h="${base_width}" d="0.01"/>

Commit message: new URDF with mesh

File: urdf/rosmower.xacro (robot description, xacro)
@@ -1,11 +1,11 @@
 <?xml version="1.0"?>
-<robot xmlns:xacro="http://www.ros.org/wiki/xacro" name="robaka_v2">
-  <xacro:property name="base_width" value="0.35"/>
+<robot xmlns:xacro="http://www.ros.org/wiki/xacro" name="HoverMower">
+  <xacro:property name="base_width" value="0.28"/>
   <xacro:property name="base_len" value="0.536"/>
-  <xacro:property name="base_height" value="0.216"/>
+  <xacro:property name="base_height" value="0.26"/>
   <xacro:property name="wheel_radius" value="0.085"/>
-  <xacro:property name="base_wheel_gap" value="-0.02"/>
-  <xacro:property name="wheel_separation" value="0.32"/>
-  <xacro:property name="wheel_joint_offset" value="-0.120"/>
+  <xacro:property name="base_wheel_gap" value="0.01"/>
+  <xacro:property name="wheel_separation" value="0.36"/>
+  <xacro:property name="wheel_joint_offset" value="0"/>
   <xacro:property name="caster_wheel_radius" value="0.035"/>
   <xacro:property name="caster_wheel_joint_offset" value="0.12"/>
@@ -37,5 +37,4 @@
     </inertial>
   </xacro:macro>
-  <link name="dummy"/>
   <link name="base_footprint">
     <xacro:box_inertia m="8" w="0.001" h="0.001" d="0.001"/>
@@ -48,8 +47,4 @@
     </visual>
   </link>
-  <joint name="dummy_joint" type="fixed">
-     <parent link="dummy"/>
-     <child link="base_footprint"/>
-     </joint>
   <link name="base_link">
     <xacro:box_inertia m="1" w="${base_len}" h="${base_width}" d="0.01"/>
@@ -57,18 +52,19 @@
       <material name="lightgray"/>
       <geometry>
-        <box size="${base_len} ${base_width} ${base_height}"/>
+        <mesh filename="package://rosmower/meshes/robot_body.dae" />
       </geometry>
     </visual>
     <collision>
       <geometry>
-        <box size="${base_len} ${base_width} ${base_height}"/>
+        <mesh filename="package://rosmower/meshes/robot_body.dae"/>
       </geometry>
     </collision>
   </link>
   <joint name="base_link_joint" type="fixed">
-    <origin xyz="0.14 0 ${wheel_radius + 0.005}" rpy="0 0 0" />
+    <origin xyz="0 0 0.08" rpy="0 0 0" />
     <parent link="base_footprint"/>
     <child link="base_link" />
   </joint>
+<!--
   <xacro:macro name="cylinder_inertia" params="m r h">
     <inertial>
@@ -77,20 +73,18 @@
     </inertial>
   </xacro:macro>
-  <xacro:macro name="wheel" params="prefix reflect">
+-->
+  <xacro:macro name="wheel" params="prefix reflect rotate">
     <link name="${prefix}_wheel">
       <visual>
-	<material name="darkgray"/>
-        <origin xyz="0 0 0" rpy="${pi/2} 0 0"/>
+        <material name="darkgray"/>
         <geometry>
-          <cylinder radius="${wheel_radius}" length="0.058"/>
+	        <mesh filename="package://rosmower/meshes/wheel.dae" />
         </geometry>
-      </visual>
-      <collision>
-        <origin xyz="0 0 0" rpy="${pi/2} 0 0"/>
-        <geometry>
-          <cylinder radius="${wheel_radius}" length="0.058"/>
-        </geometry>
-      </collision>
-      <xacro:cylinder_inertia m="10" r="${wheel_radius}" h="0.02"/>
+    </visual>
+    <collision>
+      <geometry>
+        <mesh filename="package://rosmower/meshes/wheel.dae" />
+      </geometry>
+    </collision>
     </link>
     <joint name="${prefix}_wheel" type="continuous">
@@ -98,9 +92,10 @@
       <parent link="base_link"/>
       <child link="${prefix}_wheel"/>
-      <origin xyz="${wheel_joint_offset} ${((base_width/2)+base_wheel_gap)*reflect} -0.06" rpy="0 0 0"/>
+      <origin xyz="${wheel_joint_offset} ${((base_width/2)+base_wheel_gap)*reflect} 0" rpy="0 0 ${0+rotate}"/>
     </joint>
   </xacro:macro>
-  <xacro:wheel prefix="left" reflect="1"/>
-  <xacro:wheel prefix="right" reflect="-1"/>
+  <xacro:wheel prefix="left" reflect="1" rotate="0"/>
+  <xacro:wheel prefix="right" reflect="-1" rotate="3.14159"/>
+<!--
   <xacro:macro name="sphere_inertia" params="m r">
     <inertial>
@@ -158,3 +153,4 @@
   <link name="camera_link" type="fixed">
   </link>
+  -->
 </robot>

Commit message: merge conflict

File: urdf/rosmower.xacro (robot description, xacro)
@@ -37,7 +37,4 @@
     </inertial>
   </xacro:macro>
-<<<<<<< HEAD
-=======
->>>>>>> 404f13884297039cacb8e9d9ec9f42bed27634ba
   <link name="base_footprint">
     <xacro:box_inertia m="8" w="0.001" h="0.001" d="0.001"/>
@@ -49,9 +46,5 @@
         </geometry>
     </visual>
-<<<<<<< HEAD
   </link>
-=======
-  </link>
->>>>>>> 404f13884297039cacb8e9d9ec9f42bed27634ba
   <link name="base_link">
     <xacro:box_inertia m="1" w="${base_len}" h="${base_width}" d="0.01"/>

Commit message: improve urdf with sensor links

File: urdf/rosmower.xacro (robot description, xacro)
@@ -126,8 +126,9 @@
     <origin xyz="${caster_wheel_joint_offset} 0 -${0.06+caster_wheel_radius}" rpy="0 0 0"/>
   </joint>
+-->
   <joint name="imu_joint" type="fixed">
     <parent link="base_link" />
     <child link="imu" />
-    <origin xyz="0.157 0.0 0.20" rpy="0 0 0" />
+    <origin xyz="0.092 0.0 0.105" rpy="0 0 0" />
   </joint>
   <link name="imu" />
@@ -135,22 +136,36 @@
     <parent link="base_link" />
     <child link="lidar_frame" />
-    <origin xyz="0.157 0.0 0.21" rpy="0 0 0" />
+    <origin xyz="0.242 0.0 0.195" rpy="0 0 0" />
   </joint>
-  <link name="lidar_frame">
-    <visual>
-      <material name="blue" />
-      <origin xyz="0 0 0" rpy="0 0 0"/>
-      <geometry>
-        <cylinder radius="0.032" length="0.02"/>
-      </geometry>
-    </visual>
-  </link>
+  <link name="lidar_frame" type="fixed"/>
   <joint name="camera_joint" type="fixed">
-    <origin xyz="0.185 0 0.07" rpy="0 0 3.14159" />
+    <origin xyz="0.35 0 0.117" rpy="0 0 0" />
     <parent link="base_link" />
     <child link="camera_link" />
   </joint>
-  <link name="camera_link" type="fixed">
-  </link>
-  -->
+  <link name="camera_link" type="fixed"/>
+  <joint name="perimeter_left_joint" type="fixed">
+    <origin xyz="0.385 0.081 0.025" rpy="0 0 0" />
+    <parent link="base_link" />
+    <child link="perimeter_left" />
+  </joint>
+  <link name="perimeter_left" type="fixed"/>
+  <joint name="perimeter_right_joint" type="fixed">
+    <origin xyz="0.385 -0.081 0.025" rpy="0 0 0" />
+    <parent link="base_link" />
+    <child link="perimeter_right" />
+  </joint>
+  <link name="perimeter_right" type="fixed"/>
+  <joint name="bumper_left_joint" type="fixed">
+    <origin xyz="0.45 0.101 0.040" rpy="0 0 0" />
+    <parent link="base_link" />
+    <child link="bumper_left" />
+  </joint>
+  <link name="bumper_left" type="fixed"/>
+  <joint name="bumper_right_joint" type="fixed">
+    <origin xyz="0.45 -0.101 0.040" rpy="0 0 0" />
+    <parent link="base_link" />
+    <child link="bumper_right" />
+  </joint>
+  <link name="bumper_right" type="fixed"/>
 </robot>

Commit message: operational twist_mux and move_base

File: urdf/rosmower.xacro (robot description, xacro)
@@ -29,6 +29,4 @@
     <color rgba="0.8 0.0 0.0 1.0"/>
   </material>
-  <!-- Import Rviz colors -->
-<!--  <xacro:include filename="$(find ros_robotics)/urdf/materials.xacro" /> -->
   <xacro:macro name="box_inertia" params="m w h d">
     <inertial>
@@ -66,12 +64,4 @@
     <child link="base_link" />
   </joint>
-<!--
-  <xacro:macro name="cylinder_inertia" params="m r h">
-    <inertial>
-      <mass value="${m}"/>
-      <inertia ixx="${m*(3*r*r+h*h)/12}" ixy = "0" ixz = "0" iyy="${m*(3*r*r+h*h)/12}" iyz = "0" izz="${m*r*r/2}"/>
-    </inertial>
-  </xacro:macro>
--->
   <xacro:macro name="wheel" params="prefix reflect rotate">
     <link name="${prefix}_wheel">
@@ -97,34 +87,4 @@
   <xacro:wheel prefix="left" reflect="1" rotate="0"/>
   <xacro:wheel prefix="right" reflect="-1" rotate="3.14159"/>
-<!--
-  <xacro:macro name="sphere_inertia" params="m r">
-    <inertial>
-      <mass value="${m}"/>
-      <inertia ixx="${2.0*m*(r*r)/5.0}" ixy="0.0" ixz="0.0" iyy="${2.0*m*(r*r)/5.0}" iyz="0.0" izz="${2.0*m*(r*r)/5.0}"/>
-    </inertial>
-  </xacro:macro>
-   <link name="caster_wheel">
-     <visual>
-       <material name="darkgray"/>
-      <origin xyz="0 0 0" rpy="0 0 0"/>
-      <geometry>
-        <sphere radius="${caster_wheel_radius}"/>
-      </geometry>
-    </visual>
-    <collision>
-      <origin xyz="0 0 0" rpy="0 0 0"/>
-      <geometry>
-        <sphere radius="${caster_wheel_radius}"/>
-      </geometry>
-    </collision>
-    <xacro:sphere_inertia m="5" r="${caster_wheel_radius}"/>
-  </link>
-  <joint name="caster_wheel_joint" type="continuous">
-    <axis xyz="0 1 0" rpy="0 0 0" />
-    <parent link="base_link"/>
-    <child link="caster_wheel"/>
-    <origin xyz="${caster_wheel_joint_offset} 0 -${0.06+caster_wheel_radius}" rpy="0 0 0"/>
-  </joint>
--->
   <joint name="imu_joint" type="fixed">
     <parent link="base_link" />

Commit message: remove open_mower integration because of forking it

File: urdf/rosmower.xacro (robot description, xacro)
@@ -100,4 +100,10 @@
   </joint>
   <link name="lidar_frame" type="fixed"/>
+  <joint name="gps_joint" type="fixed">
+    <parent link="base_link" />
+    <child link="gps_frame" />
+    <origin xyz="0.310 0.0 0.195" rpy="0 0 0" />
+  </joint>
+  <link name="gps_frame" type="fixed"/>
   <joint name="camera_joint" type="fixed">
     <origin xyz="0.35 0 0.117" rpy="0 0 0" />

Commit message: working robot localization with gps

File: urdf/rosmower.xacro (robot description, xacro)
@@ -103,5 +103,5 @@
     <parent link="base_link" />
     <child link="gps_frame" />
-    <origin xyz="0.310 0.0 0.195" rpy="0 0 0" />
+    <origin xyz="0.0 0.118 0.202" rpy="0 0 0" />
   </joint>
   <link name="gps_frame" type="fixed"/>

Commit message: workling robot localization

File: urdf/rosmower.xacro (robot description, xacro)
@@ -91,4 +91,5 @@
     <parent link="base_link" />
     <child link="imu" />
+ <!--   <origin xyz="0.092 0.0 0.105" rpy="0 0 -1.5708" />  -->
     <origin xyz="0.092 0.0 0.105" rpy="0 0 0" />
   </joint>
